Commit message: Exploração turbo

File: src/prm_2026/description/robot.urdf.xacro (robot description, xacro)
@@ -10,5 +10,5 @@
   <xacro:property name="wheel_ygap" value="0.025"/> <!-- Distancia entre as rodas -->
   <xacro:property name="wheel_zoff" value="0.05"/> <!-- Deslocamento da roda em Z -->
-  <xacro:property name="wheel_xoff" value="0.12"/> <!-- Deslocamento da roda em X -->
+  <xacro:property name="wheel_xoff" value="0.0"/> <!-- Rodas no eixo do centro: gira no lugar sem varrer o corpo -->
   <xacro:property name="caster_xoff" value="0.14"/> <!-- Deslocamento do caster em X -->
   <!-- Definição de algumas propriedades inerciais -->
@@ -138,4 +138,33 @@
   <!-- Very low friction on caster so it rotates freely -->
   <gazebo reference="front_caster">
+    <mu1>0.01</mu1>
+    <mu2>0.01</mu2>
+    <kp>100000.0</kp>
+    <kd>1.0</kd>
+  </gazebo>
+  <!-- Caster traseiro: com as rodas no centro, dá apoio fore/aft (não tomba). -->
+  <link name="rear_caster">
+    <visual>
+      <geometry>
+        <sphere radius="${(wheel_radius+wheel_zoff-(base_height/2))}"/>
+      </geometry>
+      <material name="DarkBlue">
+        <color rgba="0.09 0.30 0.46 1.0"/>
+      </material>
+    </visual>
+    <collision>
+      <origin xyz="0 0 0" rpy="0 0 0"/>
+      <geometry>
+        <sphere radius="${(wheel_radius+wheel_zoff-(base_height/2))}"/>
+      </geometry>
+    </collision>
+    <xacro:sphere_inertia m="0.005" r="${(wheel_radius+wheel_zoff-(base_height/2))}"/>
+  </link>
+  <joint name="rear_caster_joint" type="fixed">
+    <parent link="base_link"/>
+    <child link="rear_caster"/>
+    <origin xyz="${-caster_xoff} 0.0 ${-(base_height/2)}" rpy="0 0 0"/>
+  </joint>
+  <gazebo reference="rear_caster">
     <mu1>0.01</mu1>
     <mu2>0.01</mu2>

Commit message: Braço dinâmico v2

File: src/prm_2026/description/robot.urdf.xacro (robot description, xacro)
@@ -293,4 +293,16 @@
       <state_interface name="velocity"/>
     </joint>
+    <!-- Junta 1 (ombro/base do braço): PITCH vertical, levanta o braço 0 -> 45 graus -->
+    <joint name="shoulder_pitch">
+      <command_interface name="position">
+        <param name="min">0.0</param>
+        <param name="max">0.785398</param>
+      </command_interface>
+      <!-- Início em 0 graus: braço apontando reto para a frente -->
+      <state_interface name="position">
+        <param name="initial_value">0.0</param>
+      </state_interface>
+      <state_interface name="velocity"/>
+    </joint>
     <joint name="gripper_extension">
       <command_interface name="position">
@@ -421,5 +433,7 @@
     <parent link="base_link"/>
     <child link="camera_link"/>
-    <origin xyz="0.215 0 0.05" rpy="0 0 0"/>
+    <!-- Câmera levemente acima do plano do braço retraído (arm_base z=0.05),
+         senão o braço recolhido fica na frente da lente. -->
+    <origin xyz="0.215 0 0.085" rpy="0 0 0"/>
   </joint>
   <link name="camera_frame"/>
@@ -553,10 +567,40 @@
     </sensor> -->
   </gazebo>
-  <!-- Shoulder: sweeps arm sideways (Z-axis rotation) -->
+  <!-- Junta 1 - Ombro/base do braço: PITCH no plano vertical.
+       axis (0 -1 0): rotação positiva LEVANTA a ponta do braço.
+       lower=0 (reto para a frente), upper=0.785398 rad (45 graus). -->
+  <joint name="shoulder_pitch" type="revolute">
+    <axis xyz="0 -1 0"/>
+    <limit effort="50.0" lower="0.0" upper="0.785398" velocity="0.5"/>
+    <origin rpy="0 0 0" xyz="0.2 0 0.05"/>
+    <parent link="base_link"/>
+    <child link="arm_base"/>
+  </joint>
+  <!-- Link curto do ombro: tudo abaixo herda o pitch desta junta -->
+  <link name="arm_base">
+    <visual>
+      <geometry>
+        <cylinder length="0.04" radius="0.012"/>
+      </geometry>
+      <origin rpy="0 1.57075 0" xyz="0.02 0 0"/>
+      <material name="LightBlue">
+        <color rgba="0.11 0.37 0.56 1.0"/>
+      </material>
+    </visual>
+    <collision>
+      <geometry>
+        <cylinder length="0.04" radius="0.012"/>
+      </geometry>
+      <origin rpy="0 1.57075 0" xyz="0.02 0 0"/>
+    </collision>
+    <xacro:cylinder_inertia m="0.01" r="0.012" h="0.04"/>
+  </link>
+  <!-- Junta 2: horizontal (yaw, Z-axis), varre o braço lateralmente.
+       Re-parented para arm_base para herdar o pitch da Junta 1. -->
   <joint name="gripper_extension" type="revolute">
     <axis xyz="0 0 1"/>
     <limit effort="50.0" lower="-1.57075" upper="0.2" velocity="0.5"/>
-    <origin rpy="0 0 0" xyz="0.2 0 0.05"/>
-    <parent link="base_link"/>
+    <origin rpy="0 0 0" xyz="0.04 0 0"/>
+    <parent link="arm_base"/>
     <child link="upper_arm"/>
   </joint>

Commit message: Braço dinâmico v5

File: src/prm_2026/description/robot.urdf.xacro (robot description, xacro)
@@ -307,6 +307,6 @@
     <joint name="gripper_extension">
       <command_interface name="position">
-        <param name="min">-1.57075</param>
-        <param name="max">0.2</param>
+        <param name="min">-1.5708</param>
+        <param name="max">0.0</param>
       </command_interface>
       <!-- Início RETRAÍDO: braço recolhido contra o corpo já no spawn -->
@@ -319,5 +319,5 @@
       <command_interface name="position">
         <param name="min">-1.5708</param>
-        <param name="max">0.5</param>
+        <param name="max">0.0</param>
       </command_interface>
       <state_interface name="position">
@@ -572,5 +572,5 @@
   <joint name="shoulder_pitch" type="revolute">
     <axis xyz="0 -1 0"/>
-    <limit effort="50.0" lower="0.0" upper="0.785398" velocity="0.5"/>
+    <limit effort="50.0" lower="0.0" upper="0.785398" velocity="2.0"/>
     <origin rpy="0 0 0" xyz="0.2 0 0.05"/>
     <parent link="base_link"/>
@@ -600,5 +600,6 @@
   <joint name="gripper_extension" type="revolute">
     <axis xyz="0 0 1"/>
-    <limit effort="50.0" lower="-1.57075" upper="0.2" velocity="0.5"/>
+    <!-- Junta horizontal: amplitude limitada a 90° (-1.5708 a 0). Velocidade 2.0 (desdobra rápido). -->
+    <limit effort="50.0" lower="-1.5708" upper="0.0" velocity="2.0"/>
     <origin rpy="0 0 0" xyz="0.04 0 0"/>
     <parent link="arm_base"/>
@@ -624,5 +625,6 @@
   <joint name="arm_elbow" type="revolute">
     <axis xyz="0 0 1"/>
-    <limit effort="50.0" lower="-1.5708" upper="0.5" velocity="0.5"/>
+    <!-- Junta horizontal: amplitude limitada a 90° (-1.5708 a 0). Velocidade 2.0 (desdobra rápido). -->
+    <limit effort="50.0" lower="-1.5708" upper="0.0" velocity="2.0"/>
     <origin xyz="0.15 0 0" rpy="0 0 0"/>
     <parent link="upper_arm"/>
