Commit message: Smaller robot + fixed arm

File: description/robot.urdf.xacro (robot description, xacro)
@@ -4,5 +4,8 @@
   <!-- Definicao de Algumas Contantes -->
   <xacro:property name="base_width" value="0.31"/> <!-- Largura da base -->
-  <xacro:property name="base_length" value="0.42"/> <!-- Comprimento da base -->
+  <!-- Base QUADRADA (length = width): minimiza o raio circunscrito ao girar no
+       lugar (meia-diagonal 0.31*sqrt2/2 ~ 0.22 m vs 0.26 m da base 0.42x0.31),
+       facilitando viradas de 180 graus em corredores estreitos. -->
+  <xacro:property name="base_length" value="0.31"/> <!-- Comprimento da base -->
   <xacro:property name="base_height" value="0.18"/> <!-- Altura da base -->
   <xacro:property name="wheel_radius" value="0.10"/> <!-- Raio da roda -->
@@ -350,5 +353,5 @@
   <gazebo>
     <plugin filename="ign_ros2_control-system" name="ign_ros2_control::IgnitionROS2ControlPlugin">
-      <parameters>$(find prm_2026)/config/controller_config.yaml</parameters>
+      <parameters>$(find bb8_control)/config/controller_config.yaml</parameters>
     </plugin>
   </gazebo>

Commit message: Mudança no braço 2

File: description/robot.urdf.xacro (robot description, xacro)
@@ -14,5 +14,10 @@
   <xacro:property name="wheel_zoff" value="0.05"/> <!-- Deslocamento da roda em Z -->
   <xacro:property name="wheel_xoff" value="0.0"/> <!-- Rodas no eixo do centro: gira no lugar sem varrer o corpo -->
-  <xacro:property name="caster_xoff" value="0.14"/> <!-- Deslocamento do caster em X -->
+  <!-- Casters (rodas bobas) recuados p/ dentro da base QUADRADA 0.31 (meia=0.155):
+       0.12 dá apoio fore/aft sem ficar na beirada. -->
+  <xacro:property name="caster_xoff" value="0.12"/> <!-- Deslocamento do caster em X -->
+  <!-- Braço de junta única: comprimento ~ tamanho do robô. Mantido abaixo do
+       LIDAR (no mastro): altura máx do braço (pivô 0.10 + arm_length) < lidar. -->
+  <xacro:property name="arm_length" value="0.25"/>
   <!-- Definição de algumas propriedades inerciais -->
   <xacro:macro name="box_inertia" params="m w h d">
@@ -298,35 +303,15 @@
       <state_interface name="velocity"/>
     </joint>
-    <!-- Junta 1 (ombro/base do braço): PITCH vertical, levanta o braço 0 -> 45 graus -->
+    <!-- Braço de junta ÚNICA: PITCH vertical, amplitude 0..180°.
+         0 = à frente (nível p/ pegar a flag), 3.14159 (180°) = retraído (deitado
+         p/ trás sobre o robô), 0.785398 = erguido 45° (flag levantada). -->
     <joint name="shoulder_pitch">
       <command_interface name="position">
         <param name="min">0.0</param>
-        <param name="max">0.785398</param>
+        <param name="max">3.14159</param>
       </command_interface>
-      <!-- Início em 0 graus: braço apontando reto para a frente -->
+      <!-- Início RETRAÍDO a 180° (braço deitado p/ trás sobre o robô) -->
       <state_interface name="position">
-        <param name="initial_value">0.0</param>
-      </state_interface>
-      <state_interface name="velocity"/>
-    </joint>
-    <joint name="gripper_extension">
-      <command_interface name="position">
-        <param name="min">-1.5708</param>
-        <param name="max">0.0</param>
-      </command_interface>
-      <!-- Início RETRAÍDO em -90°: braço recolhido ao lado já no spawn. Estender
-           leva a 0 (90° de varredura) = diretamente à frente do robô. -->
-      <state_interface name="position">
-        <param name="initial_value">-1.5708</param>
-      </state_interface>
-      <state_interface name="velocity"/>
-    </joint>
-    <joint name="arm_elbow">
-      <command_interface name="position">
-        <param name="min">-1.5708</param>
-        <param name="max">0.0</param>
-      </command_interface>
-      <state_interface name="position">
-        <param name="initial_value">-1.5708</param>
+        <param name="initial_value">3.14159</param>
       </state_interface>
       <state_interface name="velocity"/>
@@ -380,8 +365,33 @@
     </visual>
   </link>
+  <!-- Mastro: ergue o LIDAR acima de todo o volume varrido pelo braço, p/ o scan
+       360° nunca ser obstruído (dispensa o scan_masker). -->
+  <link name="lidar_mast">
+    <visual>
+      <origin xyz="0 0 0.155" rpy="0 0 0"/>
+      <geometry>
+        <cylinder radius="0.012" length="0.31"/>
+      </geometry>
+      <material name="DarkBlue">
+        <color rgba="0.09 0.30 0.46 1.0"/>
+      </material>
+    </visual>
+    <collision>
+      <origin xyz="0 0 0.155" rpy="0 0 0"/>
+      <geometry>
+        <cylinder radius="0.012" length="0.31"/>
+      </geometry>
+    </collision>
+    <xacro:cylinder_inertia m="0.05" r="0.012" h="0.31"/>
+  </link>
+  <joint name="lidar_mast_joint" type="fixed">
+    <parent link="base_link"/>
+    <child link="lidar_mast"/>
+    <origin xyz="0 0 0.09" rpy="0 0 0"/>
+  </joint>
   <joint name="lidar_joint" type="fixed">
     <parent link="base_link"/>
     <child link="lidar_link"/>
-    <origin xyz="0 0 0.12" rpy="0 0 0"/>
+    <origin xyz="0 0 0.40" rpy="0 0 0"/>
   </joint>
   <gazebo reference="lidar_link">
@@ -441,7 +451,8 @@
     <parent link="base_link"/>
     <child link="camera_link"/>
-    <!-- Câmera levemente acima do plano do braço retraído (arm_base z=0.05),
-         senão o braço recolhido fica na frente da lente. -->
-    <origin xyz="0.215 0 0.085" rpy="0 0 0"/>
+    <!-- Câmera na face frontal, ABAIXO do plano do braço (pivô em z=0.16): assim o
+         braço não atrapalha a visão nem retraído (180°, p/ trás) nem estendido
+         (0°, à frente passa acima da lente). -->
+    <origin xyz="0.16 0 0.0" rpy="0 0 0"/>
   </joint>
   <link name="camera_frame"/>
@@ -575,21 +586,30 @@
     </sensor> -->
   </gazebo>
-  <!-- Junta 1 - Ombro/base do braço: PITCH no plano vertical.
-       axis (0 -1 0): rotação positiva LEVANTA a ponta do braço.
-       lower=0 (reto para a frente), upper=0.785398 rad (45 graus). -->
+  <!-- Braço de JUNTA ÚNICA: PITCH no plano vertical.
+       axis (0 -1 0): rotação positiva LEVANTA a ponta.
+         0     = à frente (horizontal, nível p/ pegar a flag)
+         pi/4  = erguido 45° (flag levantada)
+         pi    = 180°, retraído deitado p/ trás SOBRE o robô (postura inicial)
+       Pivô na frente-topo da base; comprimento ~ tamanho do robô (arm_length). -->
+  <!-- Pivô em z=0.10 (logo acima do topo do corpo 0.09): braço a 180° deita p/
+       trás sobre o corpo sem colidir. Altura máx do braço (a 90°) = 0.10+0.25 =
+       0.35 (z~0.50 do chão), ABAIXO do LIDAR no mastro (z~0.55) -> nunca obstrui
+       o scan (sem scan_masker). Grab à frente em z~0.25 do chão (mastro 0.2–0.6).
+       Damping/friction tornam o braço fisicamente amortecido (não 'voa' solto). -->
   <joint name="shoulder_pitch" type="revolute">
     <axis xyz="0 -1 0"/>
-    <limit effort="50.0" lower="0.0" upper="0.785398" velocity="2.0"/>
-    <origin rpy="0 0 0" xyz="0.2 0 0.05"/>
+    <limit effort="50.0" lower="0.0" upper="3.14159" velocity="3.0"/>
+    <origin rpy="0 0 0" xyz="0.14 0 0.10"/>
     <parent link="base_link"/>
-    <child link="arm_base"/>
-  </joint>
-  <!-- Link curto do ombro: tudo abaixo herda o pitch desta junta -->
-  <link name="arm_base">
-    <visual>
-      <geometry>
-        <cylinder length="0.04" radius="0.012"/>
-      </geometry>
-      <origin rpy="0 1.57075 0" xyz="0.02 0 0"/>
+    <child link="arm_link"/>
+    <dynamics damping="0.5" friction="0.2"/>
+  </joint>
+  <!-- Único segmento do braço (ponta = gripper) -->
+  <link name="arm_link">
+    <visual>
+      <geometry>
+        <cylinder length="${arm_length}" radius="0.012"/>
+      </geometry>
+      <origin rpy="0 1.57079 0" xyz="${arm_length/2} 0 0"/>
       <material name="LightBlue">
         <color rgba="0.11 0.37 0.56 1.0"/>
@@ -598,64 +618,15 @@
     <collision>
       <geometry>
-        <cylinder length="0.04" radius="0.012"/>
-      </geometry>
-      <origin rpy="0 1.57075 0" xyz="0.02 0 0"/>
-    </collision>
-    <xacro:cylinder_inertia m="0.01" r="0.012" h="0.04"/>
-  </link>
-  <!-- Junta 2: horizontal (yaw, Z-axis), varre o braço lateralmente.
-       Re-parented para arm_base para herdar o pitch da Junta 1. -->
-  <joint name="gripper_extension" type="revolute">
-    <axis xyz="0 0 1"/>
-    <!-- Junta horizontal: amplitude limitada a 90° (-1.5708 a 0). Velocidade 2.0 (desdobra rápido). -->
-    <limit effort="50.0" lower="-1.5708" upper="0.0" velocity="2.0"/>
-    <origin rpy="0 0 0" xyz="0.04 0 0"/>
-    <parent link="arm_base"/>
-    <child link="upper_arm"/>
-  </joint>
-  <!-- Upper arm segment (shoulder → elbow) -->
-  <link name="upper_arm">
-    <visual>
-      <geometry>
-        <cylinder length="0.15" radius="0.01"/>
-      </geometry>
-      <origin rpy="0 1.57075 0" xyz="0.075 0 0"/>
-    </visual>
-    <collision>
-      <geometry>
-        <cylinder length="0.15" radius="0.01"/>
-      </geometry>
-      <origin rpy="0 1.57075 0" xyz="0.075 0 0"/>
-    </collision>
-    <xacro:cylinder_inertia m="0.005" r="0.01" h="0.15"/>
-  </link>
-  <!-- Elbow: folds lower arm back toward body (same Z-axis rotation) -->
-  <joint name="arm_elbow" type="revolute">
-    <axis xyz="0 0 1"/>
-    <!-- Junta horizontal: amplitude limitada a 90° (-1.5708 a 0). Velocidade 2.0 (desdobra rápido). -->
-    <limit effort="50.0" lower="-1.5708" upper="0.0" velocity="2.0"/>
-    <origin xyz="0.15 0 0" rpy="0 0 0"/>
-    <parent link="upper_arm"/>
-    <child link="gripper_pole"/>
-  </joint>
-  <link name="gripper_pole">
-    <visual>
-      <geometry>
-        <cylinder length="0.2" radius="0.01"/>
-      </geometry>
-      <origin rpy="0 1.57075 0" xyz="0.1 0 0"/>
-    </visual>
-    <collision>
-      <geometry>
-        <cylinder length="0.2" radius="0.01"/>
-      </geometry>
-    </collision>
-    <xacro:cylinder_inertia m="0.01" r="0.01" h="0.2"/>
+        <cylinder length="${arm_length}" radius="0.012"/>
+      </geometry>
+      <origin rpy="0 1.57079 0" xyz="${arm_length/2} 0 0"/>
+    </collision>
+    <xacro:cylinder_inertia m="0.05" r="0.012" h="${arm_length}"/>
   </link>
   <joint name="left_gripper_joint" type="prismatic">
     <axis xyz="0 1 0"/>
     <limit effort="100.0" lower="0.0" upper="0.06" velocity="0.25"/>
-    <origin rpy="0 0 0" xyz="0.2 0.01 0"/>
-    <parent link="gripper_pole"/>
+    <origin rpy="0 0 0" xyz="${arm_length} 0.01 0"/>
+    <parent link="arm_link"/>
     <child link="left_gripper"/>
   </joint>
@@ -696,6 +667,6 @@
     <axis xyz="0 1 0"/>
     <limit effort="100.0" lower="-0.06" upper="0" velocity="0.25"/>
-    <origin rpy="0 0 0" xyz="0.2 -0.01 0"/>
-    <parent link="gripper_pole"/>
+    <origin rpy="0 0 0" xyz="${arm_length} -0.01 0"/>
+    <parent link="arm_link"/>
     <child link="right_gripper"/>
   </joint>

Commit message: Mudança no braço -> muitos bugs

File: description/robot.urdf.xacro (robot description, xacro)
@@ -4,5 +4,8 @@
   <!-- Definicao de Algumas Contantes -->
   <xacro:property name="base_width" value="0.31"/> <!-- Largura da base -->
-  <xacro:property name="base_length" value="0.42"/> <!-- Comprimento da base -->
+  <!-- Base QUADRADA (length = width): minimiza o raio circunscrito ao girar no
+       lugar (meia-diagonal 0.31*sqrt2/2 ~ 0.22 m vs 0.26 m da base 0.42x0.31),
+       facilitando viradas de 180 graus em corredores estreitos. -->
+  <xacro:property name="base_length" value="0.31"/> <!-- Comprimento da base -->
   <xacro:property name="base_height" value="0.18"/> <!-- Altura da base -->
   <xacro:property name="wheel_radius" value="0.10"/> <!-- Raio da roda -->
@@ -11,5 +14,10 @@
   <xacro:property name="wheel_zoff" value="0.05"/> <!-- Deslocamento da roda em Z -->
   <xacro:property name="wheel_xoff" value="0.0"/> <!-- Rodas no eixo do centro: gira no lugar sem varrer o corpo -->
-  <xacro:property name="caster_xoff" value="0.14"/> <!-- Deslocamento do caster em X -->
+  <!-- Casters (rodas bobas) recuados p/ dentro da base QUADRADA 0.31 (meia=0.155):
+       0.12 dá apoio fore/aft sem ficar na beirada. -->
+  <xacro:property name="caster_xoff" value="0.12"/> <!-- Deslocamento do caster em X -->
+  <!-- Braço de junta única: comprimento ~ tamanho do robô. Mantido abaixo do
+       LIDAR (no mastro): altura máx do braço (pivô 0.10 + arm_length) < lidar. -->
+  <xacro:property name="arm_length" value="0.25"/>
   <!-- Definição de algumas propriedades inerciais -->
   <xacro:macro name="box_inertia" params="m w h d">
@@ -59,5 +67,7 @@
       </geometry>
     </collision>
-    <xacro:box_inertia m="4.0" w="${base_width}" d="${base_length}" h="${base_height}"/>
+    <!-- Massa reduzida (4.0 -> 2.0 kg): menor inércia rotacional => acelera/freia
+         o giro mais rápido (viradas de 180° mais ágeis com acc_lim_theta atual). -->
+    <xacro:box_inertia m="2.0" w="${base_width}" d="${base_length}" h="${base_height}"/>
   </link>
   <!-- Definindo a Base do Robô (base footprint) -->
@@ -293,35 +303,15 @@
       <state_interface name="velocity"/>
     </joint>
-    <!-- Junta 1 (ombro/base do braço): PITCH vertical, levanta o braço 0 -> 45 graus -->
+    <!-- Braço de junta ÚNICA: PITCH vertical, amplitude 0..180°.
+         0 = à frente (nível p/ pegar a flag), 3.14159 (180°) = retraído (deitado
+         p/ trás sobre o robô), 0.785398 = erguido 45° (flag levantada). -->
     <joint name="shoulder_pitch">
       <command_interface name="position">
         <param name="min">0.0</param>
-        <param name="max">0.785398</param>
+        <param name="max">3.14159</param>
       </command_interface>
-      <!-- Início em 0 graus: braço apontando reto para a frente -->
+      <!-- Início RETRAÍDO a 180° (braço deitado p/ trás sobre o robô) -->
       <state_interface name="position">
-        <param name="initial_value">0.0</param>
-      </state_interface>
-      <state_interface name="velocity"/>
-    </joint>
-    <joint name="gripper_extension">
-      <command_interface name="position">
-        <param name="min">-1.5708</param>
-        <param name="max">0.0</param>
-      </command_interface>
-      <!-- Início RETRAÍDO em -90°: braço recolhido ao lado já no spawn. Estender
-           leva a 0 (90° de varredura) = diretamente à frente do robô. -->
-      <state_interface name="position">
-        <param name="initial_value">-1.5708</param>
-      </state_interface>
-      <state_interface name="velocity"/>
-    </joint>
-    <joint name="arm_elbow">
-      <command_interface name="position">
-        <param name="min">-1.5708</param>
-        <param name="max">0.0</param>
-      </command_interface>
-      <state_interface name="position">
-        <param name="initial_value">-1.5708</param>
+        <param name="initial_value">3.14159</param>
       </state_interface>
       <state_interface name="velocity"/>
@@ -350,5 +340,5 @@
   <gazebo>
     <plugin filename="ign_ros2_control-system" name="ign_ros2_control::IgnitionROS2ControlPlugin">
-      <parameters>$(find prm_2026)/config/controller_config.yaml</parameters>
+      <parameters>$(find bb8_control)/config/controller_config.yaml</parameters>
     </plugin>
   </gazebo>
@@ -375,8 +365,33 @@
     </visual>
   </link>
+  <!-- Mastro: ergue o LIDAR acima de todo o volume varrido pelo braço, p/ o scan
+       360° nunca ser obstruído (dispensa o scan_masker). -->
+  <link name="lidar_mast">
+    <visual>
+      <origin xyz="0 0 0.155" rpy="0 0 0"/>
+      <geometry>
+        <cylinder radius="0.012" length="0.31"/>
+      </geometry>
+      <material name="DarkBlue">
+        <color rgba="0.09 0.30 0.46 1.0"/>
+      </material>
+    </visual>
+    <collision>
+      <origin xyz="0 0 0.155" rpy="0 0 0"/>
+      <geometry>
+        <cylinder radius="0.012" length="0.31"/>
+      </geometry>
+    </collision>
+    <xacro:cylinder_inertia m="0.05" r="0.012" h="0.31"/>
+  </link>
+  <joint name="lidar_mast_joint" type="fixed">
+    <parent link="base_link"/>
+    <child link="lidar_mast"/>
+    <origin xyz="0 0 0.09" rpy="0 0 0"/>
+  </joint>
   <joint name="lidar_joint" type="fixed">
     <parent link="base_link"/>
     <child link="lidar_link"/>
-    <origin xyz="0 0 0.12" rpy="0 0 0"/>
+    <origin xyz="0 0 0.40" rpy="0 0 0"/>
   </joint>
   <gazebo reference="lidar_link">
@@ -386,9 +401,11 @@
       <always_on>true</always_on>
       <visualize>true</visualize>
-      <update_rate>20</update_rate>
+      <!-- LIDAR mais leve p/ arena pequena: 540 amostras @ 15 Hz (era 1080 @ 20 Hz).
+           Menos CPU e custmap mais responsiva; ~0.67° de resolução já é suficiente. -->
+      <update_rate>15</update_rate>
       <ray>
         <scan>
           <horizontal>
-            <samples>1080</samples>
+            <samples>540</samples>
             <resolution>1.000000</resolution>
             <min_angle>0.000000</min_angle>
@@ -434,7 +451,8 @@
     <parent link="base_link"/>
     <child link="camera_link"/>
-    <!-- Câmera levemente acima do plano do braço retraído (arm_base z=0.05),
-         senão o braço recolhido fica na frente da lente. -->
-    <origin xyz="0.215 0 0.085" rpy="0 0 0"/>
+    <!-- Câmera na face frontal, ABAIXO do plano do braço (pivô em z=0.16): assim o
+         braço não atrapalha a visão nem retraído (180°, p/ trás) nem estendido
+         (0°, à frente passa acima da lente). -->
+    <origin xyz="0.16 0 0.0" rpy="0 0 0"/>
   </joint>
   <link name="camera_frame"/>
@@ -568,21 +586,30 @@
     </sensor> -->
   </gazebo>
-  <!-- Junta 1 - Ombro/base do braço: PITCH no plano vertical.
-       axis (0 -1 0): rotação positiva LEVANTA a ponta do braço.
-       lower=0 (reto para a frente), upper=0.785398 rad (45 graus). -->
+  <!-- Braço de JUNTA ÚNICA: PITCH no plano vertical.
+       axis (0 -1 0): rotação positiva LEVANTA a ponta.
+         0     = à frente (horizontal, nível p/ pegar a flag)
+         pi/4  = erguido 45° (flag levantada)
+         pi    = 180°, retraído deitado p/ trás SOBRE o robô (postura inicial)
+       Pivô na frente-topo da base; comprimento ~ tamanho do robô (arm_length). -->
+  <!-- Pivô em z=0.10 (logo acima do topo do corpo 0.09): braço a 180° deita p/
+       trás sobre o corpo sem colidir. Altura máx do braço (a 90°) = 0.10+0.25 =
+       0.35 (z~0.50 do chão), ABAIXO do LIDAR no mastro (z~0.55) -> nunca obstrui
+       o scan (sem scan_masker). Grab à frente em z~0.25 do chão (mastro 0.2–0.6).
+       Damping/friction tornam o braço fisicamente amortecido (não 'voa' solto). -->
   <joint name="shoulder_pitch" type="revolute">
     <axis xyz="0 -1 0"/>
-    <limit effort="50.0" lower="0.0" upper="0.785398" velocity="2.0"/>
-    <origin rpy="0 0 0" xyz="0.2 0 0.05"/>
+    <limit effort="50.0" lower="0.0" upper="3.14159" velocity="3.0"/>
+    <origin rpy="0 0 0" xyz="0.14 0 0.10"/>
     <parent link="base_link"/>
-    <child link="arm_base"/>
-  </joint>
-  <!-- Link curto do ombro: tudo abaixo herda o pitch desta junta -->
-  <link name="arm_base">
-    <visual>
-      <geometry>
-        <cylinder length="0.04" radius="0.012"/>
-      </geometry>
-      <origin rpy="0 1.57075 0" xyz="0.02 0 0"/>
+    <child link="arm_link"/>
+    <dynamics damping="0.5" friction="0.2"/>
+  </joint>
+  <!-- Único segmento do braço (ponta = gripper) -->
+  <link name="arm_link">
+    <visual>
+      <geometry>
+        <cylinder length="${arm_length}" radius="0.012"/>
+      </geometry>
+      <origin rpy="0 1.57079 0" xyz="${arm_length/2} 0 0"/>
       <material name="LightBlue">
         <color rgba="0.11 0.37 0.56 1.0"/>
@@ -591,64 +618,15 @@
     <collision>
       <geometry>
-        <cylinder length="0.04" radius="0.012"/>
-      </geometry>
-      <origin rpy="0 1.57075 0" xyz="0.02 0 0"/>
-    </collision>
-    <xacro:cylinder_inertia m="0.01" r="0.012" h="0.04"/>
-  </link>
-  <!-- Junta 2: horizontal (yaw, Z-axis), varre o braço lateralmente.
-       Re-parented para arm_base para herdar o pitch da Junta 1. -->
-  <joint name="gripper_extension" type="revolute">
-    <axis xyz="0 0 1"/>
-    <!-- Junta horizontal: amplitude limitada a 90° (-1.5708 a 0). Velocidade 2.0 (desdobra rápido). -->
-    <limit effort="50.0" lower="-1.5708" upper="0.0" velocity="2.0"/>
-    <origin rpy="0 0 0" xyz="0.04 0 0"/>
-    <parent link="arm_base"/>
-    <child link="upper_arm"/>
-  </joint>
-  <!-- Upper arm segment (shoulder → elbow) -->
-  <link name="upper_arm">
-    <visual>
-      <geometry>
-        <cylinder length="0.15" radius="0.01"/>
-      </geometry>
-      <origin rpy="0 1.57075 0" xyz="0.075 0 0"/>
-    </visual>
-    <collision>
-      <geometry>
-        <cylinder length="0.15" radius="0.01"/>
-      </geometry>
-      <origin rpy="0 1.57075 0" xyz="0.075 0 0"/>
-    </collision>
-    <xacro:cylinder_inertia m="0.005" r="0.01" h="0.15"/>
-  </link>
-  <!-- Elbow: folds lower arm back toward body (same Z-axis rotation) -->
-  <joint name="arm_elbow" type="revolute">
-    <axis xyz="0 0 1"/>
-    <!-- Junta horizontal: amplitude limitada a 90° (-1.5708 a 0). Velocidade 2.0 (desdobra rápido). -->
-    <limit effort="50.0" lower="-1.5708" upper="0.0" velocity="2.0"/>
-    <origin xyz="0.15 0 0" rpy="0 0 0"/>
-    <parent link="upper_arm"/>
-    <child link="gripper_pole"/>
-  </joint>
-  <link name="gripper_pole">
-    <visual>
-      <geometry>
-        <cylinder length="0.2" radius="0.01"/>
-      </geometry>
-      <origin rpy="0 1.57075 0" xyz="0.1 0 0"/>
-    </visual>
-    <collision>
-      <geometry>
-        <cylinder length="0.2" radius="0.01"/>
-      </geometry>
-    </collision>
-    <xacro:cylinder_inertia m="0.01" r="0.01" h="0.2"/>
+        <cylinder length="${arm_length}" radius="0.012"/>
+      </geometry>
+      <origin rpy="0 1.57079 0" xyz="${arm_length/2} 0 0"/>
+    </collision>
+    <xacro:cylinder_inertia m="0.05" r="0.012" h="${arm_length}"/>
   </link>
   <joint name="left_gripper_joint" type="prismatic">
     <axis xyz="0 1 0"/>
     <limit effort="100.0" lower="0.0" upper="0.06" velocity="0.25"/>
-    <origin rpy="0 0 0" xyz="0.2 0.01 0"/>
-    <parent link="gripper_pole"/>
+    <origin rpy="0 0 0" xyz="${arm_length} 0.01 0"/>
+    <parent link="arm_link"/>
     <child link="left_gripper"/>
   </joint>
@@ -689,6 +667,6 @@
     <axis xyz="0 1 0"/>
     <limit effort="100.0" lower="-0.06" upper="0" velocity="0.25"/>
-    <origin rpy="0 0 0" xyz="0.2 -0.01 0"/>
-    <parent link="gripper_pole"/>
+    <origin rpy="0 0 0" xyz="${arm_length} -0.01 0"/>
+    <parent link="arm_link"/>
     <child link="right_gripper"/>
   </joint>
