Commit message: Robo quadrado

File: description/robot.urdf.xacro (robot description, xacro)
@@ -3,6 +3,6 @@
   xmlns:xacro="http://ros.org/wiki/xacro">
   <!-- Definicao de Algumas Contantes -->
-  <xacro:property name="base_width" value="0.31"/> <!-- Largura da base -->
-  <xacro:property name="base_length" value="0.42"/> <!-- Comprimento da base -->
+  <xacro:property name="base_width" value="0.35"/> <!-- Largura da base (corpo quadrado: == base_length) -->
+  <xacro:property name="base_length" value="0.35"/> <!-- Comprimento da base (corpo quadrado: == base_width) -->
   <xacro:property name="base_height" value="0.18"/> <!-- Altura da base -->
   <xacro:property name="wheel_radius" value="0.10"/> <!-- Raio da roda -->
@@ -59,5 +59,5 @@
       </geometry>
     </collision>
-    <xacro:box_inertia m="4.0" w="${base_width}" d="${base_length}" h="${base_height}"/>
+    <xacro:box_inertia m="2.5" w="${base_width}" d="${base_length}" h="${base_height}"/>
   </link>
   <!-- Definindo a Base do Robô (base footprint) -->
@@ -350,5 +350,9 @@
   <gazebo>
     <plugin filename="ign_ros2_control-system" name="ign_ros2_control::IgnitionROS2ControlPlugin">
-      <parameters>$(find prm_2026)/config/controller_config.yaml</parameters>
+      <!-- Config DENTRO do bb8_control (repo alvo): gripper_controller com os 5
+           joints que o gripper_server publica (shoulder_pitch, gripper_extension,
+           arm_elbow, right/left_gripper_joint). O config do prm_2026 só tinha 3
+           joints -> update() do JointGroupPositionController dava ERROR (5 != 3). -->
+      <parameters>$(find bb8_control)/config/controller_config.yaml</parameters>
     </plugin>
   </gazebo>
@@ -390,5 +394,5 @@
         <scan>
           <horizontal>
-            <samples>1080</samples>
+            <samples>360</samples>
             <resolution>1.000000</resolution>
             <min_angle>0.000000</min_angle>
@@ -398,5 +402,5 @@
         <range>
           <min>0.120000</min>
-          <max>5.0</max>
+          <max>3.5</max>
           <resolution>0.05000</resolution>
         </range>
@@ -436,5 +440,5 @@
     <!-- Câmera levemente acima do plano do braço retraído (arm_base z=0.05),
          senão o braço recolhido fica na frente da lente. -->
-    <origin xyz="0.215 0 0.085" rpy="0 0 0"/>
+    <origin xyz="0.18 0 0.085" rpy="0 0 0"/>
   </joint>
   <link name="camera_frame"/>
@@ -464,22 +468,6 @@
       <enable_metrics>true</enable_metrics>
     </sensor> -->
-    <!-- RGB camera – used by bb8_visual_slam package (rtabmap loop closure) -->
-    <sensor name="robot_cam_rgb" type="camera">
-      <topic>robot_cam_rgb</topic>
-      <camera>
-        <horizontal_fov>1.57</horizontal_fov>
-        <image>
-          <width>320</width>
-          <height>240</height>
-        </image>
-        <clip>
-          <near>0.1</near>
-          <far>100</far>
-        </clip>
-      </camera>
-      <always_on>1</always_on>
-      <update_rate>10</update_rate>
-      <visualize>false</visualize>
-    </sensor>
+    <!-- RGB camera REMOVIDA: mantida apenas a câmera semântica (corta 1 render
+         pass por frame). bb8_visual_slam (rtabmap) fica sem fonte RGB. -->
     <!-- Insere uma camera com segmentacao semantica -->
     <sensor name="robot_cam" type="segmentation">
@@ -574,5 +562,7 @@
     <axis xyz="0 -1 0"/>
     <limit effort="50.0" lower="0.0" upper="0.785398" velocity="2.0"/>
-    <origin rpy="0 0 0" xyz="0.2 0 0.05"/>
+    <!-- Realocado para o TOPO do corpo quadrado (z=base_height/2=0.09), recuado
+         do lidar central (x=0.13 > raio lidar 0.05) e à frente p/ alcançar flags. -->
+    <origin rpy="0 0 0" xyz="0.13 0 0.09"/>
     <parent link="base_link"/>
     <child link="arm_base"/>
@@ -589,10 +579,5 @@
       </material>
     </visual>
-    <collision>
-      <geometry>
-        <cylinder length="0.04" radius="0.012"/>
-      </geometry>
-      <origin rpy="0 1.57075 0" xyz="0.02 0 0"/>
-    </collision>
+    <!-- Colisão removida: elo estrutural interno, nunca toca nada. Simplifica física. -->
     <xacro:cylinder_inertia m="0.01" r="0.012" h="0.04"/>
   </link>
@@ -611,15 +596,10 @@
     <visual>
       <geometry>
-        <cylinder length="0.15" radius="0.01"/>
-      </geometry>
-      <origin rpy="0 1.57075 0" xyz="0.075 0 0"/>
-    </visual>
-    <collision>
-      <geometry>
-        <cylinder length="0.15" radius="0.01"/>
-      </geometry>
-      <origin rpy="0 1.57075 0" xyz="0.075 0 0"/>
-    </collision>
-    <xacro:cylinder_inertia m="0.005" r="0.01" h="0.15"/>
+        <cylinder length="0.10" radius="0.01"/>
+      </geometry>
+      <origin rpy="0 1.57075 0" xyz="0.05 0 0"/>
+    </visual>
+    <!-- Colisão removida: elo estrutural interno. Simplifica física. -->
+    <xacro:cylinder_inertia m="0.005" r="0.01" h="0.10"/>
   </link>
   <!-- Elbow: folds lower arm back toward body (same Z-axis rotation) -->
@@ -628,5 +608,5 @@
     <!-- Junta horizontal: amplitude limitada a 90° (-1.5708 a 0). Velocidade 2.0 (desdobra rápido). -->
     <limit effort="50.0" lower="-1.5708" upper="0.0" velocity="2.0"/>
-    <origin xyz="0.15 0 0" rpy="0 0 0"/>
+    <origin xyz="0.10 0 0" rpy="0 0 0"/>
     <parent link="upper_arm"/>
     <child link="gripper_pole"/>
@@ -635,19 +615,15 @@
     <visual>
       <geometry>
-        <cylinder length="0.2" radius="0.01"/>
-      </geometry>
-      <origin rpy="0 1.57075 0" xyz="0.1 0 0"/>
-    </visual>
-    <collision>
-      <geometry>
-        <cylinder length="0.2" radius="0.01"/>
-      </geometry>
-    </collision>
-    <xacro:cylinder_inertia m="0.01" r="0.01" h="0.2"/>
+        <cylinder length="0.12" radius="0.01"/>
+      </geometry>
+      <origin rpy="0 1.57075 0" xyz="0.06 0 0"/>
+    </visual>
+    <!-- Colisão removida: elo estrutural interno. Simplifica física. -->
+    <xacro:cylinder_inertia m="0.01" r="0.01" h="0.12"/>
   </link>
   <joint name="left_gripper_joint" type="prismatic">
     <axis xyz="0 1 0"/>
     <limit effort="100.0" lower="0.0" upper="0.06" velocity="0.25"/>
-    <origin rpy="0 0 0" xyz="0.2 0.01 0"/>
+    <origin rpy="0 0 0" xyz="0.12 0.01 0"/>
     <parent link="gripper_pole"/>
     <child link="left_gripper"/>
@@ -689,5 +665,5 @@
     <axis xyz="0 1 0"/>
     <limit effort="100.0" lower="-0.06" upper="0" velocity="0.25"/>
-    <origin rpy="0 0 0" xyz="0.2 -0.01 0"/>
+    <origin rpy="0 0 0" xyz="0.12 -0.01 0"/>
     <parent link="gripper_pole"/>
     <child link="right_gripper"/>

Commit message: Mudancas nas variaveis

File: description/robot.urdf.xacro (robot description, xacro)
@@ -402,5 +402,5 @@
         <range>
           <min>0.120000</min>
-          <max>3.5</max>
+          <max>5.0</max>
           <resolution>0.05000</resolution>
         </range>
@@ -475,5 +475,5 @@
       <camera>
         <segmentation_type>semantic</segmentation_type>
-        <horizontal_fov>1.57</horizontal_fov>
+        <horizontal_fov>1.9</horizontal_fov> <!-- FOV largo: pega a flag mais de lado durante a exploração (vision_processor.camera_hfov_deg deve casar) -->
         <image>
           <width>320</width>
@@ -561,5 +561,5 @@
   <joint name="shoulder_pitch" type="revolute">
     <axis xyz="0 -1 0"/>
-    <limit effort="50.0" lower="0.0" upper="0.785398" velocity="2.0"/>
+    <limit effort="50.0" lower="0.0" upper="0.785398" velocity="3.0"/>
     <!-- Realocado para o TOPO do corpo quadrado (z=base_height/2=0.09), recuado
          do lidar central (x=0.13 > raio lidar 0.05) e à frente p/ alcançar flags. -->
@@ -587,5 +587,5 @@
     <axis xyz="0 0 1"/>
     <!-- Junta horizontal: amplitude limitada a 90° (-1.5708 a 0). Velocidade 2.0 (desdobra rápido). -->
-    <limit effort="50.0" lower="-1.5708" upper="0.0" velocity="2.0"/>
+    <limit effort="50.0" lower="-1.5708" upper="0.0" velocity="3.0"/>
     <origin rpy="0 0 0" xyz="0.04 0 0"/>
     <parent link="arm_base"/>
@@ -607,5 +607,5 @@
     <axis xyz="0 0 1"/>
     <!-- Junta horizontal: amplitude limitada a 90° (-1.5708 a 0). Velocidade 2.0 (desdobra rápido). -->
-    <limit effort="50.0" lower="-1.5708" upper="0.0" velocity="2.0"/>
+    <limit effort="50.0" lower="-1.5708" upper="0.0" velocity="3.0"/>
     <origin xyz="0.10 0 0" rpy="0 0 0"/>
     <parent link="upper_arm"/>

Commit message: Comentários

File: description/robot.urdf.xacro (robot description, xacro)
@@ -704,3 +704,19 @@
     <xacro:box_inertia m="0.005" w="0.01" h="0.01" d="0.06"/>
   </link>
+  <!-- Alto atrito + contato rígido nos dedos/pontas da garra: segura a haste da
+       flag firme, sem escorregar (a flag é leve, então atrito alto resolve). -->
+  <xacro:macro name="grip_friction" params="ref">
+    <gazebo reference="${ref}">
+      <mu1>200.0</mu1>
+      <mu2>200.0</mu2>
+      <kp>1e6</kp>
+      <kd>1.0</kd>
+      <minDepth>0.001</minDepth>
+      <maxVel>0.0</maxVel>
+    </gazebo>
+  </xacro:macro>
+  <xacro:grip_friction ref="left_gripper"/>
+  <xacro:grip_friction ref="right_gripper"/>
+  <xacro:grip_friction ref="left_tip"/>
+  <xacro:grip_friction ref="right_tip"/>
 </robot>
